File: mouse.kicad_pcb (KiCad board)
At the start: 2 copper layers, 96.5 x 96.5 mm, 70 parts, among them J1 Conn_01x08_Male, J2 Conn_01x04_Male, J3 Conn_01x02_Male, J4 Conn_01x06_Male, J5 Conn_01x06_Male, Q1 Q_NPN_BCE, SW1 SW_DIP_x01, SW2 SW_SPDT, SW3 SW_SPDT, U1 LBR-127HLD, U10 LBR-127HLD, U11 STM32F303K8Tx, U12 MPU6050, U13 NJM7805SDL1, U14 XBEE_MODULE, U15 TB6612FNG, U2 LBR-127HLD, U3 LBR-127HLD, U4 LBR-127HLD, U5 LBR-127HLD, U6 LBR-127HLD, U7 LBR-127HLD, U8 LBR-127HLD, U9 LBR-127HLD

Commit message: fix: シルクの修正
Parts:
- U1, U10, U2, U3, U4, U5, U6, U7, U8, U9: footprint MyFootprint:LBR-127HLD -> MyFootprint:LBR-127HLD_2
