File: mouse.sch (KiCad schematic (older format))
At the start: 54 parts, among them J1 Conn_01x08_Male, J2 Conn_01x04_Male, J3 Conn_01x02_Male, J4 Conn_01x06_Male, J5 Conn_01x06_Male, Q1 Q_NPN_BCE, SW1 SW_DIP_x01, SW2 SW_SPDT, SW3 SW_SPDT, U1 LBR-127HLD, U10 LBR-127HLD, U11 STM32F303K8Tx, U12 MPU6050, U13 NJM7805SDL1, U14 XBEE_MODULE, U15 TB6612FNG, U2 LBR-127HLD, U3 LBR-127HLD, U4 LBR-127HLD, U5 LBR-127HLD, U6 LBR-127HLD, U7 LBR-127HLD, U8 LBR-127HLD, U9 LBR-127HLD

Commit message: fix: シルクの修正
Parts:
- U1, U10, U2, U3, U4, U5, U6, U7, U8, U9: footprint MyFootprint:LBR-127HLD -> MyFootprint:LBR-127HLD_2
Changed lines of the file:
@@
 F 0 "U2" H 1350 5575 50  0000 C CNN
 F 1 "LBR-127HLD" H 1350 5484 50  0000 C CNN
-F 2 "MyFootprint:LBR-127HLD" H 1350 5250 50  0001 C CNN
+F 2 "MyFootprint:LBR-127HLD_2" H 1350 5250 50  0001 C CNN
 F 3 "" H 1350 5250 50  0001 C CNN
 	1    1350 5250
@@
 F 0 "U4" H 1350 6575 50  0000 C CNN
 F 1 "LBR-127HLD" H 1350 6484 50  0000 C CNN
-F 2 "MyFootprint:LBR-127HLD" H 1350 6250 50  0001 C CNN
+F 2 "MyFootprint:LBR-127HLD_2" H 1350 6250 50  0001 C CNN
 F 3 "" H 1350 6250 50  0001 C CNN
 	1    1350 6250
@@
 F 0 "U6" H 1350 7625 50  0000 C CNN
 F 1 "LBR-127HLD" H 1350 7534 50  0000 C CNN
-F 2 "MyFootprint:LBR-127HLD" H 1350 7300 50  0001 C CNN
+F 2 "MyFootprint:LBR-127HLD_2" H 1350 7300 50  0001 C CNN
 F 3 "" H 1350 7300 50  0001 C CNN
 	1    1350 7300
@@
 F 0 "U8" H 1450 8675 50  0000 C CNN
 F 1 "LBR-127HLD" H 1450 8584 50  0000 C CNN
-F 2 "MyFootprint:LBR-127HLD" H 1450 8350 50  0001 C CNN
+F 2 "MyFootprint:LBR-127HLD_2" H 1450 8350 50  0001 C CNN
 F 3 "" H 1450 8350 50  0001 C CNN
 	1    1450 8350
@@
 F 0 "U10" H 1450 9775 50  0000 C CNN
 F 1 "LBR-127HLD" H 1450 9684 50  0000 C CNN
-F 2 "MyFootprint:LBR-127HLD" H 1450 9450 50  0001 C CNN
+F 2 "MyFootprint:LBR-127HLD_2" H 1450 9450 50  0001 C CNN
 F 3 "" H 1450 9450 50  0001 C CNN
 	1    1450 9450
@@
 F 0 "U1" H 1350 5575 50  0000 C CNN
 F 1 "LBR-127HLD" H 1350 5484 50  0000 C CNN
-F 2 "MyFootprint:LBR-127HLD" H 1350 5250 50  0001 C CNN
+F 2 "MyFootprint:LBR-127HLD_2" H 1350 5250 50  0001 C CNN
 F 3 "" H 1350 5250 50  0001 C CNN
 	1    1350 5250
@@
 F 0 "U9" H 1450 9775 50  0000 C CNN
 F 1 "LBR-127HLD" H 1450 9684 50  0000 C CNN
-F 2 "MyFootprint:LBR-127HLD" H 1450 9450 50  0001 C CNN
+F 2 "MyFootprint:LBR-127HLD_2" H 1450 9450 50  0001 C CNN
 F 3 "" H 1450 9450 50  0001 C CNN
 	1    1450 9450
@@
 F 0 "U3" H 1350 6575 50  0000 C CNN
 F 1 "LBR-127HLD" H 1350 6484 50  0000 C CNN
-F 2 "MyFootprint:LBR-127HLD" H 1350 6250 50  0001 C CNN
+F 2 "MyFootprint:LBR-127HLD_2" H 1350 6250 50  0001 C CNN
 F 3 "" H 1350 6250 50  0001 C CNN
 	1    1350 6250
@@
 F 0 "U5" H 1350 7625 50  0000 C CNN
 F 1 "LBR-127HLD" H 1350 7534 50  0000 C CNN
-F 2 "MyFootprint:LBR-127HLD" H 1350 7300 50  0001 C CNN
+F 2 "MyFootprint:LBR-127HLD_2" H 1350 7300 50  0001 C CNN
 F 3 "" H 1350 7300 50  0001 C CNN
 	1    1350 7300
@@
 F 0 "U7" H 1450 8675 50  0000 C CNN
 F 1 "LBR-127HLD" H 1450 8584 50  0000 C CNN
-F 2 "MyFootprint:LBR-127HLD" H 1450 8350 50  0001 C CNN
+F 2 "MyFootprint:LBR-127HLD_2" H 1450 8350 50  0001 C CNN
 F 3 "" H 1450 8350 50  0001 C CNN
 	1    1450 8350
